File: RotoPD.kicad_sch (KiCad schematic)
At the start: 43 parts, among them IC5 TPS62933DRLR, IC6 AP33772SDKZ-13-FA01, J6 10172013-00011LF, Q1 BSS138, Q2 BSS138, U10 AON7262E, U11 AON7262E, U6 TVS2200DRV, U7 TPD1E05U06DPY, U8 TPD1E05U06DPY, U9 TVS2200DRV

Commit message: changes
Parts:
- removed J6: 10172013-00011LF, 1017201300011LF, symbol USB_C_16P:10172013-00011LF
- removed L1: 10uH, 74439370100, symbol 74439370100:74439370100
- removed R15: 61.9k, Resistor_SMD:R_0603_1608Metric, symbol Device:R
- added C25: 33nF, Capacitor_SMD:C_1206_3216Metric, symbol Device:C
- added C26: 10uF, Capacitor_SMD:C_0603_1608Metric, symbol Device:C
- added IC17: XC6220B331ER-G, Library:XC6220B331ERG, symbol XC6220B331ER-G:XC6220B331ER-G
- added J16: UJ20-C-H-G-SMT-5-P16-TR, Library:UJ20CHGSMT5P16TR, symbol UJ20-C-H-G-SMT-5-P16-TR:UJ20-C-H-G-SMT-5-P16-TR
- added L2: SRP1250-7R8M, Library:SRP12507R8M, symbol SRP1250-7R8M:SRP1250-7R8M
- D2: footprint ESD122DMYR -> Library:ESD122DMYR
- IC5: footprint SOTFL50P160X60-8N -> Library:SOTFL50P160X60-8N
- IC6: footprint AP33772SDKZ13FA01 -> Library:AP33772SDKZ13FA01
Connections:
- net MNET is gone; now on net +5V: C14.1, Cout1.1, Rfbt1.1
- net +5V: now also C26.2, IC17.3 (CE), IC17.5 (VIN_1), IC17.6 (VIN_2), L2.2; no longer Cout1.2, Rfbb1.2
- net CC1: now also J16.A5 (CC1)
- net CC2: now also J16.B5 (CC2)
- net GND: now also C9.1, Cout1.2, Rfbb1.2, C25.2, C26.1, IC17.4 (VSS), IC17.7 (EP), J16.A1 (GND_1), J16.B1 (GND_2), J16.MP1, J16.MP2, J16.MP3, J16.MP4; no longer C9.2
- net USB_N: now also J16.A7 (DN1), J16.B7 (DN2)
- net USB_P: now also J16.A6 (DP1), J16.B6 (DP2)
- net VBUS: now also J16.A4 (VBUS_1), J16.B4 (VBUS_2)
- net VCC: now also C9.2, C25.1; no longer C9.1
- net at C11.2, IC5.5 (SW): now also L2.1
- new net +3V3: IC17.1 (VOUT_1), IC17.2 (VOUT_2)
- no-connect marks 12 -> 13
Other:
- note added: "Line Control"
- note added: "PD Sink"
- note added: "USB AND ESD"
- moved on the sheet: C10, C11, C12, C13, C14, C15, C16, C17, C18, C9, Cout1, D2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
