File: USB_CONTROL.kicad_sch (KiCad schematic)
At the start: 8 parts, among them J11 10172013-00011LF, U6 TVS2200DRV, U7 TPD1E05U06DPY, U8 TPD1E05U06DPY, U9 TVS2200DRV

Commit message: small changes
Parts:
- renumbered D4 to D1, J11 to J5, R31 to R12, R32 to R13, U6 to U2, U7 to U3, U8 to U4, U9 to U5
Changed lines of the file:
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@@
 		(on_board yes)
 		(dnp no)
-		(property "Reference" "#PWR078"
+		(property "Reference" "#PWR032"
 			(at 177.8 134.62 0)
 			(effects
@@
 			(project "first_project"
 				(path "/2e03126f-90c3-49c2-bb02-7889a4a780ce/c3f59fbc-6924-4e8b-96b8-62bdd14c37a6"
-					(reference "#PWR078")
+					(reference "#PWR032")
 					(unit 1)
 				)
@@
 		(dnp no)
 		(fields_autoplaced yes)
-		(property "Reference" "R31"
+		(property "Reference" "R12"
 			(at 95.25 114.2999 0)
 			(effects
@@
 			(project "first_project"
 				(path "/2e03126f-90c3-49c2-bb02-7889a4a780ce/c3f59fbc-6924-4e8b-96b8-62bdd14c37a6"
-					(reference "R31")
+					(reference "R12")
 					(unit 1)
 				)
@@
 		(dnp no)
 		(fields_autoplaced yes)
-		(property "Reference" "#PWR075"
+		(property "Reference" "#PWR029"
 			(at 153.67 123.19 0)
 			(effects
@@
 			(project "first_project"
 				(path "/2e03126f-90c3-49c2-bb02-7889a4a780ce/c3f59fbc-6924-4e8b-96b8-62bdd14c37a6"
-					(reference "#PWR075")
+					(reference "#PWR029")
 					(unit 1)
 				)
@@
 		(dnp no)
 		(fields_autoplaced yes)
-		(property "Reference" "U9"
+		(property "Reference" "U5"
 			(at 213.36 101.5999 0)
 			(effects
@@
 			(project "first_project"
 				(path "/2e03126f-90c3-49c2-bb02-7889a4a780ce/c3f59fbc-6924-4e8b-96b8-62bdd14c37a6"
-					(reference "U9")
+					(reference "U5")
 					(unit 1)
 				)
@@
 		(dnp no)
 		(fields_autoplaced yes)
-		(property "Reference" "#PWR076"
+		(property "Reference" "#PWR030"
 			(at 177.8 118.11 0)
 			(effects
@@
 			(project ""
 				(path "/2e03126f-90c3-49c2-bb02-7889a4a780ce/c3f59fbc-6924-4e8b-96b8-62bdd14c37a6"
-					(reference "#PWR076")
+					(reference "#PWR030")
 					(unit 1)
 				)
@@
 		(dnp no)
 		(fields_autoplaced yes)
-		(property "Reference" "#PWR080"
+		(property "Reference" "#PWR034"
 			(at 209.55 116.84 0)
 			(effects
@@
 			(project "first_project"
 				(path "/2e03126f-90c3-49c2-bb02-7889a4a780ce/c3f59fbc-6924-4e8b-96b8-62bdd14c37a6"
-					(reference "#PWR080")
+					(reference "#PWR034")
 					(unit 1)
 				)
@@
 		(dnp no)
 		(fields_autoplaced yes)
-		(property "Reference" "U6"
+		(property "Reference" "U2"
 			(at 181.61 102.8699 0)
 			(effects
@@
 			(project ""
 				(path "/2e03126f-90c3-49c2-bb02-7889a4a780ce/c3f59fbc-6924-4e8b-96b8-62bdd14c37a6"
-					(reference "U6")
+					(reference "U2")
 					(unit 1)
 				)
@@
 		(dnp no)
 		(fields_autoplaced yes)
-		(property "Reference" "#PWR079"
+		(property "Reference" "#PWR033"
 			(at 193.04 130.81 0)
 			(effects
@@
 			(project ""
 				(path "/2e03126f-90c3-49c2-bb02-7889a4a780ce/c3f59fbc-6924-4e8b-96b8-62bdd14c37a6"
-					(reference "#PWR079")
+					(reference "#PWR033")
 					(unit 1)
 				)
@@
 		(dnp no)
 		(fields_autoplaced yes)
-		(property "Reference" "J11"
+		(property "Reference" "J5"
 			(at 124.46 88.9 0)
 			(effects
@@
 			(project "first_project"
 				(path "/2e03126f-90c3-49c2-bb02-7889a4a780ce/c3f59fbc-6924-4e8b-96b8-62bdd14c37a6"
-					(reference "J11")
+					(reference "J5")
 					(unit 1)
 				)
@@
 		(dnp no)
 		(fields_autoplaced yes)
-		(property "Reference" "#PWR073"
+		(property "Reference" "#PWR027"
 			(at 99.06 88.9 0)
 			(effects
@@
 			(project "first_project"
 				(path "/2e03126f-90c3-49c2-bb02-7889a4a780ce/c3f59fbc-6924-4e8b-96b8-62bdd14c37a6"
-					(reference "#PWR073")
+					(reference "#PWR027")
 					(unit 1)
 				)
@@
 		(dnp no)
 		(fields_autoplaced yes)
-		(property "Reference" "U8"
+		(property "Reference" "U4"
 			(at 173.99 144.7799 90)
 			(effects
@@
 			(project "first_project"
 				(path "/2e03126f-90c3-49c2-bb02-7889a4a780ce/c3f59fbc-6924-4e8b-96b8-62bdd14c37a6"
-					(reference "U8")
+					(reference "U4")
 					(unit 1)
 				)
@@
 		(dnp no)
 		(fields_autoplaced yes)
-		(property "Reference" "R32"
+		(property "Reference" "R13"
 			(at 156.21 111.7599 0)
 			(effects
@@
 			(project "first_project"
 				(path "/2e03126f-90c3-49c2-bb02-7889a4a780ce/c3f59fbc-6924-4e8b-96b8-62bdd14c37a6"
-					(reference "R32")
+					(reference "R13")
 					(unit 1)
 				)
@@
 		(dnp no)
 		(fields_autoplaced yes)
-		(property "Reference" "#PWR072"
+		(property "Reference" "#PWR026"
 			(at 97.79 125.73 0)
 			(effects
@@
 			(project "first_project"
 				(path "/2e03126f-90c3-49c2-bb02-7889a4a780ce/c3f59fbc-6924-4e8b-96b8-62bdd14c37a6"
-					(reference "#PWR072")
+					(reference "#PWR026")
 					(unit 1)
 				)
@@
 		(dnp no)
 		(fields_autoplaced yes)
-		(property "Reference" "D4"
+		(property "Reference" "D1"
 			(at 214.63 123.19 0)
 			(effects
@@
 			(project ""
 				(path "/2e03126f-90c3-49c2-bb02-7889a4a780ce/c3f59fbc-6924-4e8b-96b8-62bdd14c37a6"
-					(reference "D4")
+					(reference "D1")
 					(unit 1)
 				)
@@
 		(dnp no)
 		(fields_autoplaced yes)
-		(property "Reference" "U7"
+		(property "Reference" "U3"
 			(at 173.99 129.5399 90)
 			(effects
@@
 			(project ""
 				(path "/2e03126f-90c3-49c2-bb02-7889a4a780ce/c3f59fbc-6924-4e8b-96b8-62bdd14c37a6"
-					(reference "U7")
+					(reference "U3")
 					(unit 1)
 				)
@@
 		(dnp no)
 		(fields_autoplaced yes)
-		(property "Reference" "#PWR077"
+		(property "Reference" "#PWR031"
 			(at 177.8 119.38 0)
 			(effects
@@
 			(project ""
 				(path "/2e03126f-90c3-49c2-bb02-7889a4a780ce/c3f59fbc-6924-4e8b-96b8-62bdd14c37a6"
-					(reference "#PWR077")
+					(reference "#PWR031")
 					(unit 1)
 				)
@@
 		(dnp no)
 		(fields_autoplaced yes)
-		(property "Reference" "#PWR074"
+		(property "Reference" "#PWR028"
 			(at 153.67 90.17 0)
 			(effects
@@
 			(project "first_project"
 				(path "/2e03126f-90c3-49c2-bb02-7889a4a780ce/c3f59fbc-6924-4e8b-96b8-62bdd14c37a6"
-					(reference "#PWR074")
-					(unit 1)
-				)
+					(reference "#PWR028")
+					(unit 1)
+				)

Commit message: changes
Parts:
- removed J5: 10172013-00011LF, 1017201300011LF, symbol USB_C_16P:10172013-00011LF
- added J5: UJ20-C-H-G-SMT-5-P16-TR, Library:UJ20CHGSMT5P16TR, symbol UJ20-C-H-G-SMT-5-P16-TR:UJ20-C-H-G-SMT-5-P16-TR
- D1: footprint ESD122DMYR -> Library:ESD122DMYR
Connections:
- net CC1: now also J5.A5 (CC1)
- net CC2: now also J5.B5 (CC2)
- net D+: now also J5.A6 (DP1), J5.B6 (DP2)
- net D-: now also J5.A7 (DN1), J5.B7 (DN2)
- net GND: now also J5.A1 (GND_1), J5.B1 (GND_2), J5.MP1, J5.MP2, J5.MP3, J5.MP4
- net VBUS: now also J5.A4 (VBUS_1), J5.B4 (VBUS_2)
Other:
- moved on the sheet: R12, R13
