File: first_project.kicad_pcb (KiCad board)
At the start: 2 copper layers, 129.1 x 55 mm, 99 parts, among them IC1 MCP1416T-E_OT, IC10 INA226AIDGSR, IC11 MCP1416T-E_OT, IC12 INA226AIDGSR, IC13 MCP1416T-E_OT, IC14 INA226AIDGSR, IC2 INA226AIDGSR, IC3 MAX31865ATP+T, IC4 NAU7802SGI, IC5 MAX31865ATP+T, IC6 MAX31865ATP+T, IC7 MAX31865ATP+T, IC8 AP33772DKZ-13, IC9 MCP1416T-E_OT, J1 NTMFS5C612NLT1G, J10 1757242, J11 10172013-00011LF, J12 NTMFS5C612NLT1G, J13 1757242, J14 NTMFS5C612NLT1G, J15 1757242, J2 1757242, J3 B4B-XH-A_LF__SN_, J4 B4B-XH-A_LF__SN_, J5 B4B-XH-A_LF__SN_, J6 B4B-XH-A_LF__SN_, J7 B4B-XH-A_LF__SN_, J8 10172013-00011LF, J9 NTMFS5C612NLT1G, U1 ESP32-S3-MINI-1, U2 TVS2200DRV, U3 TPD1E05U06DPY, U4 TPD1E05U06DPY, U5 TVS2200DRV, U6 TVS2200DRV, U7 TPD1E05U06DPY, U8 TPD1E05U06DPY, U9 TVS2200DRV

Commit message: small changes
Parts:
- removed the C12 at (120.6, 134.4)
- removed the IC3 at (179.3, 123.8)
- removed the IC6 at (209.3, 123.8)
- removed the J5 at (200.5, 145.0)
- removed the J6 at (215.5, 145.0)
- removed the R10 at (185.0, 127.0)
- removed the R11 at (186.5, 127.0)
- removed the R14 at (215.0, 127.0)
- removed the R16 at (230.0, 127.0)
- removed the R17 at (231.5, 127.0)
- removed the S1 at (182.0, 135.0)
- removed the U6 at (115.1, 107.6)
- added C10: 100nF, Capacitor_SMD:C_1206_3216Metric, F.Cu at (91.8, 43.7)
- added C17: 1u, Capacitor_SMD:C_0603_1608Metric, F.Cu at (105.7, 104.8)
- added C18: 100nF, Capacitor_SMD:C_0402_1005Metric, F.Cu at (106.4, 100.6)
- added C19: 100nF, Capacitor_SMD:C_0402_1005Metric, F.Cu at (147.9, 134.3)
- added C20: 4.7uF, Capacitor_SMD:C_1206_3216Metric, F.Cu at (141.6, 125.0)
- added C21: 100nF, Capacitor_SMD:C_0402_1005Metric, F.Cu at (131.7, 134.3)
- added C22: 4.7uF, Capacitor_SMD:C_1206_3216Metric, F.Cu at (125.4, 125.0)
- added C23: 100nF, Capacitor_SMD:C_0402_1005Metric, F.Cu at (115.6, 134.4)
- added C24: 4.7uF, Capacitor_SMD:C_1206_3216Metric, F.Cu at (109.3, 125.1)
- added Cout1: 100uF, Capacitor_SMD:C_1206_3216Metric, F.Cu at (99.5, 45.2)
- added D1: ESD122DMYR, Library:ESD122DMYR, F.Cu at (161.5, 106.7)
- added D2: ESD122DMYR, Library:ESD122DMYR, F.Cu at (93.1, 107.5)
- added D4: D_Schottky, Diode_SMD:D_SMA, F.Cu at (118.0, 104.8)
- added IC14: MCP1416T-E_OT, Library:SOT95P270X145-5N, F.Cu at (104.8, 122.5)
- added IC15: INA226AIDGSR, Library:SOP50P490X110-10N, F.Cu at (116.3, 130.6)
- added IC5: TPS62933DRLR, Library:SOTFL50P160X60-8N, F.Cu at (93.8, 48.8)
- added J10: NTMFS5C612NLT1G, Library:NTMFS5C612NLT1G, F.Cu at (138.7, 130.7)
- added J15: 1757242, Library:1757242, F.Cu at (107.9, 138.2)
- added Q1: BSS138, Package_TO_SOT_SMD:SOT-323_SC-70, F.Cu at (118.2, 98.2)
- added Q2: BSS138, Package_TO_SOT_SMD:SOT-323_SC-70, F.Cu at (118.2, 100.8)
- added R21: 5.1k, Resistor_SMD:R_0402_1005Metric, F.Cu at (120.5, 98.1)
- added R22: 5.1k, Resistor_SMD:R_0402_1005Metric, F.Cu at (120.5, 100.8)
- added R23: 5.1k, Resistor_SMD:R_0402_1005Metric, F.Cu at (114.7, 99.6)
- added R25: 5.1k, Resistor_SMD:R_0402_1005Metric, F.Cu at (111.4, 97.7)
- added R26: 10k, Resistor_SMD:R_0402_1005Metric, F.Cu at (109.8, 97.7)
- added R41: 10k, Resistor_SMD:R_0402_1005Metric, F.Cu at (120.8, 125.7)
- added R42: 10k, Resistor_SMD:R_0402_1005Metric, F.Cu at (119.2, 125.3)
- added R45: 10k, Resistor_SMD:R_0402_1005Metric, F.Cu at (132.7, 125.4)
- added R47: 30mΩ, Resistor_SMD:R_2512_6332Metric, F.Cu at (112.4, 131.1)
- added R48: 10k, Resistor_SMD:R_0402_1005Metric, F.Cu at (104.7, 125.8)
- added R49: 10k, Resistor_SMD:R_0402_1005Metric, F.Cu at (103.1, 125.4)
- added R50: 10k, Resistor_SMD:R_0402_1005Metric, F.Cu at (106.3, 125.4)
- added R51: 10k, Resistor_SMD:R_0402_1005Metric, F.Cu at (117.6, 125.5)
- added R52: 10k, Resistor_SMD:R_0402_1005Metric, F.Cu at (116.6, 125.5)
- added R53: 10k, Resistor_SMD:R_0402_1005Metric, F.Cu at (115.5, 125.5)
- added Rfbb1: 10k, Resistor_SMD:R_1206_3216Metric, F.Cu at (97.0, 45.1)
- added Rfbt1: 52.3k, Resistor_SMD:R_1206_3216Metric, F.Cu at (102.0, 46.8)
- added S2: 219-4MST, Library:2194MST, F.Cu at (174.4, 129.5)
- added TH1: Thermistor_NTC, Resistor_SMD:R_0402_1005Metric, F.Cu at (106.3, 99.5)
- added U10: AON7262E, Library:TRANS_AONR21307, F.Cu at (107.5, 108.7)
- added U11: AON7262E, Library:TRANS_AONR21307, F.Cu at (111.3, 108.7)
- added U8: TPD1E05U06DPY, Package_SON:Texas_DPY0002A_0.6x1mm_P0.65mm, F.Cu at (91.9, 106.3)
- C11: footprint Capacitor_SMD:C_0402_1005Metric -> Capacitor_SMD:C_1206_3216Metric
- C12: renamed from C17; value 4.7uF -> 10u
- C13: value 4.7uF -> 33nF
- C14: value 100nF -> 15pF; footprint Capacitor_SMD:C_0402_1005Metric -> Capacitor_SMD:C_1206_3216Metric
- C15: value 4.7uF -> 10u
- C9: value 1uF -> 10uF; footprint Capacitor_SMD:C_0402_1005Metric -> Capacitor_SMD:C_1206_3216Metric
- D3: renamed from D4; value ESD122DMYR -> RED; footprint Library:ESD122DMYR -> LED_SMD:LED_0603_1608Metric
- D5: renamed from D3; value ESD122DMYR -> RED; footprint Library:ESD122DMYR -> LED_SMD:LED_0603_1608Metric
- IC10, IC12: value INA226AIDGSR -> MCP1416T-E_OT; footprint Library:SOP50P490X110-10N -> Library:SOT95P270X145-5N
- IC11, IC13: value MCP1416T-E_OT -> INA226AIDGSR; footprint Library:SOT95P270X145-5N -> Library:SOP50P490X110-10N
- IC6: renamed from IC14; value INA226AIDGSR -> AP33772SDKZ-13-FA01; footprint Library:SOP50P490X110-10N -> Library:AP33772SDKZ13FA01
- IC8: value AP33772DKZ-13 -> MAX31865ATP+T; footprint Library:QFN50P400X400X80-25N-D -> Library:QFN65P500X500X80-21N
- IC9: value MCP1416T-E_OT -> MAX31865ATP+T; footprint Library:SOT95P270X145-5N -> Library:QFN65P500X500X80-21N
- J11: value 10172013-00011LF -> 1757242; footprint Library:1017201300011LF -> Library:1757242
- J3, J4, J7: value B4B-XH-A_LF__SN_ -> 691412120004B; footprint Library:B4BXHALFSN -> Library:691412120004B
- J5: renamed from J10; value 1757242 -> 10172013-00011LF; footprint Library:1757242 -> Library:1017201300011LF
- J6: renamed from J15; value 1757242 -> 10172013-00011LF; footprint Library:1757242 -> Library:1017201300011LF
- J8: value 10172013-00011LF -> 691412120004B; footprint Library:1017201300011LF -> Library:691412120004B
- J9: value NTMFS5C612NLT1G -> 691412120004B; footprint Library:NTMFS5C612NLT1G -> Library:691412120004B
- R12: renamed from R25; value 10k -> 5.1k
- R13: renamed from R26; value 10k -> 5.1k
- R14: renamed from R41; value 10k -> 5.1k
- R15: value 4.3k -> 61.9k; footprint Resistor_SMD:R_0402_1005Metric -> Resistor_SMD:R_0603_1608Metric
- R16: renamed from R42; value 10k -> 5.1k
- R17: renamed from R45; value 10k -> 5m; footprint Resistor_SMD:R_0402_1005Metric -> Resistor_SMD:R_0805_2012Metric
- R18: value 150k -> 27R
- R19: value 10mR -> 10k
- R20: value 10k -> 5.1k
- R24: value 30mΩ -> 5.1k; footprint Resistor_SMD:R_2512_6332Metric -> Resistor_SMD:R_0402_1005Metric
- R27, R29: value 10k -> 430
- R28, R30: value 10k -> 4.3k
- R31: value 5.1k -> 430
- R32: value 5.1k -> 4.3k
- U6: renamed from U8; value TPD1E05U06DPY -> TVS2200DRV; footprint Package_SON:Texas_DPY0002A_0.6x1mm_P0.65mm -> Package_SON:WSON-6-1EP_2x2mm_P0.65mm_EP1x1.6mm
- moved R15 146.1 mm to (95.0, 45.9), turned to -90 degrees
- moved C14 112.5 mm to (97.5, 49.0), turned to 180 degrees
- moved U6 97.9 mm to (98.5, 106.5), turned to 180 degrees
- moved J9 97.8 mm to (208.9, 141.4), turned to 0 degrees
- moved IC9 95.7 mm to (204.5, 118.3), turned to 90 degrees
- moved R32 90.8 mm to (211.7, 121.5)
- moved R31 87.8 mm to (210.2, 121.5)
- moved D5 84.9 mm to (114.9, 97.6), turned to 180 degrees
- moved C13 75.5 mm to (96.7, 51.7)
- moved IC8 74.9 mm to (188.2, 118.3)
- moved R30 74.4 mm to (195.3, 121.5)
- moved J6 74.0 mm to (93.6, 99.8)
- moved R29 71.9 mm to (193.8, 121.5)
- moved J7 70.7 mm to (159.8, 141.4), turned to 0 degrees
- moved C9 69.0 mm to (91.8, 46.2), turned to 180 degrees
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- renumbered IC4 to IC3, IC5 to IC4, R12 to R10, R13 to R11, S2 to S1
Connections:
- C11 pad 1: Net-(IC8-IFB) -> Net-(IC5-BST)
- C11 pad 2: GND -> Net-(IC5-SW)
- C12 pad 1: VCC -> /PD/VBUS_SENSED
- C13 pad 1: VCC -> GND
- C13 pad 2: GND -> Net-(IC5-SS)
- C14 pad 1: +3V3 -> /PD/MNET
- C14 pad 2: GND -> Net-(IC5-FB)
- C15 pad 1: VCC -> /PD/VCC
- C16 pad 1: +3V3 -> /PD/IFB
- C5 pad 1: Net-(IC4-AVDD/LDO) -> Net-(IC3-AVDD/LDO)
- C8 pad 1: Net-(IC4-AVDD/LDO) -> Net-(IC3-AVDD/LDO)
- C9 pad 1: /USBPD/VBUS -> /PD/VCC
- D3 pad 2: /D- -> Net-(D3-A)
- D5 pad 2: /USBPD/D+ -> Net-(D5-A)
- IC10 pad 1: Net-(IC10-A1) -> unconnected-(IC10-NC-Pad1)
- IC10 pad 2: Net-(IC10-A0) -> +3V3
- IC10 pad 3: Net-(IC10-ALERT) -> /HEATER_PWM_2
- IC10 pad 4: /SDA -> GND
- IC10 pad 5: /SCL -> Net-(IC10-OUT)
- IC11 pad 1: unconnected-(IC11-NC-Pad1) -> Net-(IC11-A1)
- IC11 pad 2: +3V3 -> Net-(IC11-A0)
- IC11 pad 3: /HEATER_PWM_4 -> Net-(IC11-ALERT)
- IC11 pad 4: GND -> /SDA
- IC11 pad 5: Net-(IC11-OUT) -> /SCL
- IC12 pad 1: Net-(IC12-A1) -> unconnected-(IC12-NC-Pad1)
- IC12 pad 2: Net-(IC12-A0) -> +3V3
- IC12 pad 3: Net-(IC12-ALERT) -> /HEATER_PWM_3
- IC12 pad 4: /SDA -> GND
- IC12 pad 5: /SCL -> Net-(IC12-OUT)
- IC13 pad 1: unconnected-(IC13-NC-Pad1) -> Net-(IC13-A1)
- IC13 pad 2: +3V3 -> Net-(IC13-A0)
- IC13 pad 3: /HEATER_PWM_4 -> Net-(IC13-ALERT)
- IC13 pad 4: GND -> /SDA
- IC13 pad 5: Net-(IC13-OUT) -> /SCL
- IC3 pad 1: Net-(IC4-AVDD/LDO) -> Net-(IC3-AVDD/LDO)
- IC3 pad 16: Net-(IC4-AVDD/LDO) -> Net-(IC3-AVDD/LDO)
- IC3 pad 2: Net-(IC4-VIN1N) -> Net-(IC3-VIN1N)
- IC3 pad 3: Net-(IC4-VIN1P) -> Net-(IC3-VIN1P)
- IC6 pad 1: Net-(IC14-A1) -> /PD/VBUS
- IC6 pad 10: VCC -> unconnected-(IC6-NC_3-Pad10)
- IC6 pad 2: Net-(IC14-A0) -> unconnected-(IC6-NC_1-Pad2)
- IC6 pad 3: Net-(IC14-ALERT) -> GND
- IC6 pad 4: /SDA -> /PD/SDA_5V
- IC6 pad 5: /SCL -> /PD/SCL_5V
- IC6 pad 6: +3V3 -> unconnected-(IC6-FLIP-Pad6)
- IC6 pad 7: GND -> unconnected-(IC6-NC_2-Pad7)
- IC6 pad 8: VCC -> /PD/PD_LED
- IC6 pad 9: /Heater_Mosfet_4/IN- -> /PD/PD_INT_5V
- IC7 pad 13: /SS3 -> /SS2
- IC7 pad 3: /Temp Sensor 4/ISENSOR -> /Temp Sensor 2/ISENSOR
- IC7 pad 4: /Temp Sensor 4/ISENSOR -> /Temp Sensor 2/ISENSOR
- IC7 pad 5: /Temp Sensor 4/FORCE_P -> /Temp Sensor 2/FORCE_P
- IC7 pad 7: /Temp Sensor 4/RTDIN_P -> /Temp Sensor 2/RTDIN_P
- IC7 pad 8: /Temp Sensor 4/RTDIN_N -> /Temp Sensor 2/RTDIN_N
- IC7 pad 9: /Temp Sensor 4/FORCE_N -> /Temp Sensor 2/FORCE_N
- IC8 pad 1: /USBPD/VBUS -> Net-(IC8-BIAS)
- IC8 pad 10: unconnected-(IC8-NC_2-Pad10) -> GND
- IC8 pad 11: unconnected-(IC8-GPIO5-Pad11) -> /MOSI
- IC8 pad 12: unconnected-(IC8-V3VD-Pad12) -> /SCK
- IC8 pad 13: unconnected-(IC8-OTP-Pad13) -> /SS3
- IC8 pad 14: unconnected-(IC8-VFB-Pad14) -> /MISO
- IC8 pad 15: Net-(IC8-IFB) -> GND
- IC8 pad 16: /USBPD/CC2 -> GND
- IC8 pad 17: /USBPD/CC1 -> unconnected-(IC8-N.C.-Pad17)
- IC8 pad 19: unconnected-(IC8-NC_4-Pad19) -> +3V3
- IC8 pad 2: unconnected-(IC8-NC_1-Pad2) -> Net-(IC8-BIAS)
- IC8 pad 20: +5V -> +3V3
- IC8 pad 21: unconnected-(IC8-NC_5-Pad21) -> GND
- IC8 pad 3: GND -> /Temp Sensor 3/ISENSOR
- IC8 pad 4: /SDA -> /Temp Sensor 3/ISENSOR
- IC8 pad 5: /SCL -> /Temp Sensor 3/FORCE_P
- IC8 pad 6: /USBPD/FAULT -> GND
- IC8 pad 7: unconnected-(IC8-GPIO2-Pad7) -> /Temp Sensor 3/RTDIN_P
- IC8 pad 8: unconnected-(IC8-GPIO1-Pad8) -> /Temp Sensor 3/RTDIN_N
- IC8 pad 9: unconnected-(IC8-GPIO3-Pad9) -> /Temp Sensor 3/FORCE_N
- IC9 pad 1: unconnected-(IC9-NC-Pad1) -> Net-(IC9-BIAS)
- IC9 pad 2: +3V3 -> Net-(IC9-BIAS)
- IC9 pad 3: /HEATER_PWM_2 -> /Temp Sensor 4/ISENSOR
- IC9 pad 4: GND -> /Temp Sensor 4/ISENSOR
- IC9 pad 5: Net-(IC9-OUT) -> /Temp Sensor 4/FORCE_P
- J11 pad 1: GND -> /Heater_Mosfet_2/OUT_MOS
- J11 pad 2: GND -> /Heater_Mosfet_2/IN-
- J13 pad 1: /Heater_Mosfet_3/IN- -> /Heater_Mosfet_3/OUT_MOS
- J13 pad 2: /Heater_Mosfet_3/OUT_MOS -> /Heater_Mosfet_3/IN-
- J2 pad 1: /Heater_Mosfet_1/IN- -> /Heater_Mosfet_1/OUT_MOS
- J2 pad 2: /Heater_Mosfet_1/OUT_MOS -> /Heater_Mosfet_1/IN-
- J3 pad 1: /Temp Sensor 2/FORCE_N -> Net-(IC3-AVDD/LDO)
- J3 pad 2: /Temp Sensor 2/RTDIN_N -> GND
- J3 pad 3: /Temp Sensor 2/RTDIN_P -> Net-(IC3-VIN1N)
- J3 pad 4: /Temp Sensor 2/FORCE_P -> Net-(IC3-VIN1P)
- J4 pad 1: Net-(IC4-VIN1P) -> /Temp Sensor 2/FORCE_P
- J4 pad 2: Net-(IC4-VIN1N) -> /Temp Sensor 2/RTDIN_P
- J4 pad 3: GND -> /Temp Sensor 2/RTDIN_N
- J4 pad 4: Net-(IC4-AVDD/LDO) -> /Temp Sensor 2/FORCE_N
- J5 pad 1: /Heater_Mosfet_2/IN- -> GND
- J5 pad 2: /Heater_Mosfet_2/OUT_MOS -> GND
- J6 pad 1: /Heater_Mosfet_4/IN- -> GND
- J6 pad 2: /Heater_Mosfet_4/OUT_MOS -> GND
- J7 pad 1: /Temp Sensor 4/FORCE_N -> /Temp Sensor 1/FORCE_P
- J7 pad 2: /Temp Sensor 4/RTDIN_N -> /Temp Sensor 1/RTDIN_P
- J7 pad 3: /Temp Sensor 4/RTDIN_P -> /Temp Sensor 1/RTDIN_N
- J7 pad 4: /Temp Sensor 4/FORCE_P -> /Temp Sensor 1/FORCE_N
- J8 pad 1: GND -> /Temp Sensor 3/FORCE_P
- J8 pad 2: GND -> /Temp Sensor 3/RTDIN_P
- J8 pad 3: GND -> /Temp Sensor 3/RTDIN_N
- J8 pad 4: GND -> /Temp Sensor 3/FORCE_N
- J9 pad 1: Net-(J9-S_1) -> /Temp Sensor 4/FORCE_P
- J9 pad 2: Net-(J9-S_1) -> /Temp Sensor 4/RTDIN_P
- J9 pad 3: Net-(J9-S_1) -> /Temp Sensor 4/RTDIN_N
- J9 pad 4: Net-(J9-G) -> /Temp Sensor 4/FORCE_N
- R12 pad 1: Net-(IC9-OUT) -> /USB_CONTROL/CC1
- R12 pad 2: Net-(R25-Pad2) -> GND
- R13 pad 1: Net-(IC9-OUT) -> /USB_CONTROL/CC2
- R13 pad 2: Net-(J9-G) -> GND
- R14 pad 1: Net-(IC13-OUT) -> /PD/CC1
- R14 pad 2: Net-(R41-Pad2) -> GND
- R15 pad 1: /Temp Sensor 3/4300R -> GND
- R16 pad 1: Net-(IC13-OUT) -> /PD/CC2
- R16 pad 2: Net-(J14-G) -> GND
- R17 pad 1: Net-(IC14-A0) -> /PD/VBUS
- R17 pad 2: GND -> /PD/VBUS_SENSED
- R18 pad 1: /USBPD/VBUS -> /PD/VOUT
- R18 pad 2: Net-(D1-A) -> /PD/VCC
- R19 pad 1: /USBPD/VBUS -> /PD/VCC
- R19 pad 2: VCC -> Net-(D3-A)
- R20 pad 1: /USBPD/FAULT -> /PD/PD_LED
- R20 pad 2: Net-(D2-A) -> Net-(D5-A)
- R24 pad 1: /Heater_Mosfet_2/IN- -> /PD/V5V
- R24 pad 2: VCC -> /PD/SDA_5V
- R27 pad 1: Net-(R25-Pad2) -> /Temp Sensor 2/430R
- R27 pad 2: Net-(J9-S_1) -> Net-(IC7-BIAS)
- R28 pad 1: Net-(IC10-A1) -> /Temp Sensor 2/4300R
- R28 pad 2: GND -> Net-(IC7-BIAS)
- R29 pad 1: Net-(IC10-A0) -> /Temp Sensor 3/430R
- R29 pad 2: GND -> Net-(IC8-BIAS)
- R30 pad 1: Net-(IC10-ALERT) -> /Temp Sensor 3/4300R
- R30 pad 2: +3V3 -> Net-(IC8-BIAS)
- R31 pad 1: /USB_CONTROL/CC1 -> /Temp Sensor 4/430R
- R31 pad 2: GND -> Net-(IC9-BIAS)
- R32 pad 1: /USB_CONTROL/CC2 -> /Temp Sensor 4/4300R
- R32 pad 2: GND -> Net-(IC9-BIAS)
- R33 pad 1: /Heater_Mosfet_3/IN- -> /Heater_Mosfet_2/IN-
- R34 pad 1: Net-(IC11-OUT) -> Net-(IC10-OUT)
- R35 pad 1: Net-(IC11-OUT) -> Net-(IC10-OUT)
- R35 pad 2: Net-(J12-G) -> Net-(J10-G)
- R36 pad 2: Net-(J12-S_1) -> Net-(J10-S_1)
- R37 pad 1: Net-(IC12-A1) -> Net-(IC11-A1)
- R38 pad 1: Net-(IC12-A0) -> Net-(IC11-A0)
- R39 pad 1: Net-(IC12-ALERT) -> Net-(IC11-ALERT)
- R40 pad 1: /Heater_Mosfet_4/IN- -> /Heater_Mosfet_3/IN-
- R43 pad 2: Net-(J14-S_1) -> Net-(J12-S_1)
- R44 pad 1: Net-(IC14-A1) -> Net-(IC13-A1)
- R46 pad 1: Net-(IC14-ALERT) -> Net-(IC13-ALERT)
- U2 pad 4: /USBPD/VBUS -> /USB_CONTROL/VBUS
- U2 pad 5: /USBPD/VBUS -> /USB_CONTROL/VBUS
- U2 pad 6: /USBPD/VBUS -> /USB_CONTROL/VBUS
- U3 pad 1: /USBPD/CC1 -> /USB_CONTROL/CC1
- U4 pad 1: /USBPD/CC2 -> /USB_CONTROL/CC2
- U5 pad 4: /USBPD/VBUS -> /USB_CONTROL/VBUS
- U5 pad 5: /USBPD/VBUS -> /USB_CONTROL/VBUS
- U5 pad 6: /USBPD/VBUS -> /USB_CONTROL/VBUS
- U6 pad 1: /USB_CONTROL/CC2 -> GND
- U7 pad 1: /USB_CONTROL/CC1 -> /PD/CC1
- U9 pad 4: /USB_CONTROL/VBUS -> /PD/VBUS
- U9 pad 5: /USB_CONTROL/VBUS -> /PD/VBUS
- U9 pad 6: /USB_CONTROL/VBUS -> /PD/VBUS
Routing:
- net /MOSI: track 79.4 -> 0.00 mm, vias 4 -> 0
- net /SCK: track 76.4 -> 0.00 mm, vias 4 -> 0
- net /MISO: track 73.9 -> 0.00 mm, vias 5 -> 0
- net /D-: track 40.7 -> 0.15 mm
- net /D+: track 38.4 -> 0.15 mm, vias 2 -> 0
- net /PD/CC2: track 0.00 -> 27.2 mm, vias 0 -> 2
- net /SDA: track 0.00 -> 25.5 mm
- net /SCL: track 0.00 -> 25.0 mm
- net /LDCL_SDIO: track 28.6 -> 4.24 mm, vias 2 -> 1
- net /LDCL_DRDY: track 28.2 -> 3.90 mm, vias 2 -> 1
- net /LDCL_SCLK: track 28.4 -> 4.07 mm, vias 2 -> 1
- net /PD/CC1: track 0.00 -> 23.9 mm, vias 0 -> 1
- net /PD/VBUS_SENSED: track 0.00 -> 17.2 mm, vias 0 -> 2
- net /PD/V5V: track 0.00 -> 16.7 mm, vias 0 -> 3
- net GND: track 32.8 -> 16.9 mm, vias 13 -> 1
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- added copper zone on B.Cu, net /PD/VBUS
- added copper zone on F.Cu, net /PD/VBUS
- added copper zone on F.Cu, net /PD/VCC
- removed copper zone on F.Cu, net /USBPD/VBUS
Other:
- board size 129.1 x 55 mm -> 130.1 x 52.5 mm
- copper layers 2 -> 4

Commit message: changes
Parts:
- removed J6: 10172013-00011LF, Library:1017201300011LF
- removed R15: 61.9k, Resistor_SMD:R_0603_1608Metric
- removed U1: ESP32-S3-MINI-1, RF_Module:ESP32-S2-MINI-1
- added C25: 33nF, Capacitor_SMD:C_1206_3216Metric, F.Cu at (110.5, 105.5)
- added C26: 10uF, Capacitor_SMD:C_0603_1608Metric, F.Cu at (116.5, 114.0)
- added H1: MountingHole_Pad, MountingHole:MountingHole_3.2mm_M3_Pad_Via, F.Cu at (148.1, 118.4)
- added H2: MountingHole_Pad, MountingHole:MountingHole_3.2mm_M3_Pad_Via, F.Cu at (103.4, 92.0)
- added H3: MountingHole_Pad, MountingHole:MountingHole_3.2mm_M3_Pad_Via, F.Cu at (149.8, 92.3)
- added H4: MountingHole_Pad, MountingHole:MountingHole_3.2mm_M3_Pad_Via, F.Cu at (187.7, 92.3)
- added H5: MountingHole_Pad, MountingHole:MountingHole_3.2mm_M3_Pad_Via, F.Cu at (211.9, 111.5)
- added IC16: ESP32-S3-MINI-1-N8, Library:ESP32S3MINI1N8, F.Cu at (136.4, 96.5)
- added IC17: XC6220B331ER-G, Library:XC6220B331ERG, F.Cu at (116.1, 110.5)
- added J16: UJ20-C-H-G-SMT-5-P16-TR, Library:UJ20CHGSMT5P16TR, F.Cu at (93.6, 91.9)
- added L2: SRP1250-7R8M, Library:SRP12507R8M, F.Cu at (94.5, 111.5)
- J5: value 10172013-00011LF -> UJ20-C-H-G-SMT-5-P16-TR; footprint Library:1017201300011LF -> Library:UJ20CHGSMT5P16TR
- moved Rfbt1 71.7 mm to (108.8, 118.1), turned to 0 degrees
- moved Cout1 71.1 mm to (110.3, 115.5), turned to 0 degrees
- moved Rfbb1 69.2 mm to (110.3, 113.0), turned to 0 degrees
- moved C9 67.0 mm to (110.5, 110.5)
- moved C10 67.0 mm to (110.5, 108.0), turned to 0 degrees
- moved C14 65.2 mm to (106.5, 113.6), turned to 90 degrees
- moved IC5 62.4 mm to (106.7, 109.9), turned to 180 degrees
- moved C13 61.3 mm to (104.0, 112.5), turned to 90 degrees
- moved C11 57.2 mm to (104.0, 107.6), turned to 90 degrees
- moved C16 12.0 mm to (107.1, 89.8), turned to 90 degrees
- moved C18 11.1 mm to (109.1, 89.8), turned to 90 degrees
- moved TH1 9.80 mm to (108.1, 89.8), turned to 90 degrees
- moved U4 8.48 mm to (159.2, 98.1)
- moved U3 8.45 mm to (162.4, 98.1)
- moved R13 8.41 mm to (158.2, 98.2)
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Connections:
- C14 pad 1: /PD/MNET -> +5V
- C9 pad 1: /PD/VCC -> GND
- C9 pad 2: GND -> /PD/VCC
- Cout1 pad 1: /PD/MNET -> +5V
- Cout1 pad 2: +5V -> GND
- IC5 pad 1: Net-(IC5-RT) -> unconnected-(IC5-RT-Pad1)
- Rfbb1 pad 2: +5V -> GND
- Rfbt1 pad 1: /PD/MNET -> +5V
Routing:
- net /SCK: track 0.00 -> 98.6 mm, vias 0 -> 2
- net /MISO: track 0.00 -> 97.8 mm, vias 0 -> 4
- net /MOSI: track 0.00 -> 93.9 mm, vias 0 -> 4
- net /SCL: track 25.0 -> 115.5 mm, vias 0 -> 4
- net /SDA: track 25.5 -> 110.8 mm, vias 0 -> 4
- net /SS4: track 0.00 -> 78.5 mm, vias 0 -> 2
- net /SS3: track 0.00 -> 63.0 mm, vias 0 -> 2
- net /HEATER_PWM_1: track 0.00 -> 54.4 mm, vias 0 -> 2
- net /LDCL_SDIO: track 4.24 -> 53.3 mm, vias 1 -> 2
- net /LDCL_SCLK: track 4.07 -> 53.1 mm, vias 1 -> 2
- net /LDCL_DRDY: track 3.90 -> 52.8 mm, vias 1 -> 2
- net /SS2: track 0.00 -> 47.8 mm, vias 0 -> 2
- net /D-: track 0.15 -> 41.5 mm
- net /HEATER_PWM_4: track 0.00 -> 41.0 mm
- net /D+: track 0.15 -> 40.7 mm
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- added copper zone on F.Cu, net +5V
- added copper zone on F.Cu, net Net-(IC5-BST)
- added copper zone on F.Cu, net Net-(IC5-FB)
- added copper zone on F.Cu, net Net-(IC5-SS)
- added copper zone on F.Cu, net Net-(IC5-SW)
Other:
- board size 130.1 x 52.5 mm -> 130.1 x 60.5 mm
