File: first_project.kicad_sch (KiCad schematic)
At the start: 8 parts, among them J1 USB_C_Receptacle_USB2.0_16P, U1 ESP32-S3-MINI-1

Commit message: Added stuff
Parts:
- removed J1: USB_C_Receptacle_USB2.0_16P, symbol Connector:USB_C_Receptacle_USB2.0_16P
- removed R3, R4: 5.1k, symbol Device:R
Connections:
- net FAN_PWM renamed LDCL_DRDY
- net HX717_DOUT renamed LDCL_SDIO
- net HX717_SCK renamed LDCL_SCLK
- no-connect marks 4 -> 1
Other:
- sheet Heater_Mosfet renamed Heater_Mosfet_1
- removed sheet PT100
- added sheet Heater_Mosfet_2 (HEATER.kicad_sch)
- added sheet Heater_Mosfet_3 (HEATER.kicad_sch)
- added sheet Heater_Mosfet_4 (HEATER.kicad_sch)
- added sheet Temp Sensor 1 (PT100.kicad_sch)
- added sheet Temp Sensor 2 (PT100.kicad_sch)
- added sheet Temp Sensor 3 (PT100.kicad_sch)
- added sheet Temp Sensor 4 (PT100.kicad_sch)
- added sheet USB_CONTROL (USB_CONTROL.kicad_sch)
- added sheet USBPD (USBPD.kicad_sch)
- sheet Loadcell_Amplifier ports: added DRDY, SCLK, SDIO; removed none
- moved on the sheet: C1, C2, R1, R2, U1

Commit message: small changes
Other:
- removed sheet USBPD
- added sheet PD (RotoPD.kicad_sch)
- moved on the sheet: C1, C2, R1, R2, U1

Commit message: changes
Parts:
- removed U1: ESP32-S3-MINI-1, RF_Module:ESP32-S2-MINI-1, symbol RF_Module:ESP32-S3-MINI-1
- added H1, H2, H3, H4, H5: MountingHole_Pad, MountingHole:MountingHole_3.2mm_M3_Pad_Via, symbol Mechanical:MountingHole_Pad
- added IC16: ESP32-S3-MINI-1-N8, Library:ESP32S3MINI1N8, symbol ESP32-S3-MINI-1-N8-C:ESP32-S3-MINI-1-N8
Connections:
- net +3V3: now also IC16.3 (3V3)
- net ALERT_INTERRUPT: now also IC16.10 (IO6)
- net BOOT: now also IC16.4 (IO0)
- net D+: now also IC16.24 (IO20)
- net D-: now also IC16.23 (IO19)
- net ENABLE: now also IC16.45 (EN)
- net GND: now also H1.1, H2.1, H3.1, H4.1, H5.1, IC16.1 (GND_1), IC16.2 (GND_2), IC16.42 (GND_3), IC16.43 (GND_4), IC16.46 (GND_5), IC16.47 (GND_6), IC16.48 (GND_7), IC16.49 (GND_8), IC16.50 (GND_9), IC16.51 (GND_10), IC16.52 (GND_11), IC16.53 (GND_12), IC16.54 (GND_13), IC16.55 (GND_14), IC16.56 (GND_15), IC16.57 (GND_16), IC16.58 (GND_17), IC16.59 (GND_18), IC16.60 (GND_19), IC16.61 (GND_20), IC16.62 (GND_21), IC16.63 (GND_22), IC16.64 (GND_23), IC16.65 (GND_24), IC16.66 (GND_25), IC16.67 (GND_26), IC16.68 (GND_27), IC16.69 (GND_28), IC16.70 (GND_29), IC16.71 (GND_30), IC16.72 (GND_31), IC16.73 (GND_32)
- net HEATER_PWM_1: now also IC16.5 (IO1)
- net HEATER_PWM_2: now also IC16.9 (IO5)
- net HEATER_PWM_3: now also IC16.8 (IO4)
- net HEATER_PWM_4: now also IC16.6 (IO2)
- net LCD_BL: now also IC16.25 (IO21)
- net LCD_CS: now also IC16.22 (IO18)
- net LCD_SCL: now also IC16.21 (IO17)
- net LCD_SDA: now also IC16.20 (IO16)
- net LDCL_DRDY: now also IC16.32 (IO36)
- net LDCL_SCLK: now also IC16.31 (IO35)
- net LDCL_SDIO: now also IC16.30 (IO48)
- net MISO: now also IC16.13 (IO9)
- net MOSI: now also IC16.15 (IO11)
- net SCK: now also IC16.14 (IO10)
- net SCL: now also IC16.11 (IO7)
- net SDA: now also IC16.12 (IO8)
- net SS1: now also IC16.16 (IO12)
- net SS2: now also IC16.17 (IO13)
- net SS3: now also IC16.18 (IO14)
- net SS4: now also IC16.19 (IO15)
- net TP_IRQ: now also IC16.29 (IO34)
- net TP_RST: now also IC16.28 (IO33)
- net TP_SCL: now also IC16.27 (IO47)
- net TP_SDA: now also IC16.26 (IO26)
- no-connect marks 1 -> 0
