File: HEATER.kicad_sch (KiCad schematic)
At the start: 13 parts, among them IC1 INA226AIDGSR, IC2 MCP1416T-E_OT, J2 NTMFS5C612NLT1G, J3 1757242

Commit message: Added stuff
Parts:
- IC1: renamed from IC2; footprint SOT95P270X145-5N -> Library:SOT95P270X145-5N
- IC2: renamed from IC1; footprint SOP50P490X110-10N -> Library:SOP50P490X110-10N
- J1: renamed from J2; footprint NTMFS5C612NLT1G -> Library:NTMFS5C612NLT1G
- J2: renamed from J3; footprint 1757242 -> Library:1757242
- renumbered C4 to C3, C3 to C4, R8 to R3, R7 to R4, R9 to R7, R10 to R8, R11 to R9
Connections:
- net +3V3: now also R9.2
- net GND: now also R7.2, R8.2
- net VCC: now also IC2.10 (IN+), R3.2
- net IN-: now reaches J2.1
- net IN-: now also IC2.9 (IN-), R3.1
- net OUT_MOS: now reaches J1.5 (D_1), J1.6 (D_2), J1.7 (D_3), J1.8 (D_4), J1.9 (D_5), J2.2

Commit message: small changes
Connections:
- net IN-: now also J2.2; no longer J2.1
- net OUT_MOS: now also J2.1; no longer J2.2
Other:
- moved on the sheet: J2

Commit message: lots of change
Parts:
- removed J2: 1757242, Library:1757242, symbol Phoenix 5.08 2P:1757242
- added J2: 691322310002, Library:691322310002, symbol afterburner_symbolic:691322310002
Connections:
- net IN-: now also J2.2
- net OUT_MOS: now also J2.1
- net ALERT_INT: now reaches IC2.3 (ALERT), R9.1
Changed lines of the file:
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@@
+		)
+	)
+	(hierarchical_label "ALERT_INT"
+		(shape input)
+		(at 194.31 115.57 0)
+		(effects
+			(font
+				(size 1.27 1.27)
+			)
+			(justify left)
 		)
 	)
@@
 	)
 	(symbol
-		(lib_id "Phoenix 5.08 2P:1757242")
-		(at 189.23 55.88 180)
-		(unit 1)
-		(exclude_from_sim no)
-		(in_bom yes)
-		(on_board yes)
-		(dnp no)
-		(property "Reference" "J2"
-			(at 172.72 55.8801 0)
-			(effects
-				(font
-					(size 1.27 1.27)
-				)
-				(justify left)
-			)
-		)
-		(property "Value" "1757242"
-			(at 172.72 53.3401 0)
-			(effects
-				(font
-					(size 1.27 1.27)
-				)
-				(justify left)
-			)
-		)
-		(property "Footprint" "Library:1757242"
-			(at 172.72 -39.04 0)
-			(effects
-				(font
-					(size 1.27 1.27)
-				)
-				(justify left top)
-				(hide yes)
-			)
-		)
-		(property "Datasheet" "http://www.phoenixcontact.com/de/produkte/1757242/pdf"
-			(at 172.72 -139.04 0)
-			(effects
-				(font
-					(size 1.27 1.27)
-				)
-				(justify left top)
-				(hide yes)
-			)
-		)
-		(property "Description" "PCB header, nominal cross section: 2.5 mm?, color: green, nominal current: 12 A, rated voltage (III/2): 320 V, contact surface: Tin, type of contact: Male connector, Number of potentials: 2, Number of rows: 1, Number of positions per row: 2, number of connections: 2, product range: MSTBA 2,5/..-G, pitch: 5.08 mm, mounting: Wave soldering, pin layout: Linear pinning, solder pin [P]: 3.5 mm, Stecksystem: CLASSIC COMBICON, Locking: without, type of packaging: packed in cardboard"
-			(at 189.23 55.88 0)
-			(effects
-				(font
-					(size 1.27 1.27)
-				)
-				(hide yes)
-			)
-		)
-		(property "Height" "8.72"
-			(at 172.72 -339.04 0)
-			(effects
-				(font
-					(size 1.27 1.27)
-				)
-				(justify left top)
-				(hide yes)
-			)
-		)
-		(property "Mouser Part Number" "651-1757242"
-			(at 172.72 -439.04 0)
-			(effects
-				(font
-					(size 1.27 1.27)
-				)
-				(justify left top)
-				(hide yes)
-			)
-		)
-		(property "Mouser Price/Stock" "https://www.mouser.co.uk/ProductDetail/Phoenix-Contact/1757242?qs=uD%2FdkN7XIa3Ejiz9qDxlzw%3D%3D"
-			(at 172.72 -539.04 0)
-			(effects
-				(font
-					(size 1.27 1.27)
-				)
-				(justify left top)
-				(hide yes)
-			)
-		)
-		(property "Manufacturer_Name" "Phoenix Contact"
-			(at 172.72 -639.04 0)
-			(effects
-				(font
-					(size 1.27 1.27)
-				)
-				(justify left top)
-				(hide yes)
-			)
-		)
-		(property "Manufacturer_Part_Number" "1757242"
-			(at 172.72 -739.04 0)
-			(effects
-				(font
-					(size 1.27 1.27)
-				)
-				(justify left top)
-				(hide yes)
-			)
-		)
-		(pin "2"
-		)
-		(pin "1"
-		)
-		(instances
-			(project "first_project"
-				(path "/2e03126f-90c3-49c2-bb02-7889a4a780ce/7dcf5a40-78e3-4718-8bc4-f9cdc266173a"
-					(reference "J2")
-					(unit 1)
-				)
-				(path "/2e03126f-90c3-49c2-bb02-7889a4a780ce/a445d34f-af0c-4abc-8750-cad3f5a4f178"
-					(reference "J13")
-					(unit 1)
-				)
-				(path "/2e03126f-90c3-49c2-bb02-7889a4a780ce/e44134ae-6fd5-457c-b7e1-8d10f2737c1e"
-					(reference "J15")
-					(unit 1)
-				)
-				(path "/2e03126f-90c3-49c2-bb02-7889a4a780ce/f4b37abd-93fa-47ac-8113-341753863783"
-					(reference "J11")
-					(unit 1)
-				)
-			)
-		)
-	)
-	(symbol
 		(lib_id "Device:R")
 		(at 148.59 83.82 90)
@@
 					(unit 1)
 				)
+			)
+		)
+	)
+	(symbol
+		(lib_id "afterburner_symbolic:691322310002")
+		(at 184.15 53.34 90)
+		(unit 1)
+		(exclude_from_sim no)
+		(in_bom yes)
+		(on_board yes)
+		(dnp no)
+		(fields_autoplaced yes)
+		(property "Reference" "J2"
+			(at 185.42 46.99 90)
+			(effects
+				(font
+					(size 1.27 1.27)
+				)
+			)
+		)
+		(property "Value" "691322310002"
+			(at 185.42 49.53 90)
+			(effects
+				(font
+					(size 1.27 1.27)
+				)
+			)
+		)
+		(property "Footprint" "Library:691322310002"
+			(at 184.15 53.34 0)
+			(effects
+				(font
+					(size 1.27 1.27)
+				)
+				(justify bottom)
+				(hide yes)
+			)
+		)
+		(property "Datasheet" ""
+			(at 184.15 53.34 0)
+			(effects
+				(font
+					(size 1.27 1.27)
+				)
+				(hide yes)
+			)
+		)
+		(property "Description" ""
+			(at 184.15 53.34 0)
+			(effects
+				(font
+					(size 1.27 1.27)
+				)
+				(hide yes)
+			)
+		)
+		(pin "1"
+		)
+		(pin "2"
+		)
+		(instances
+			(project ""
+				(path "/2e03126f-90c3-49c2-bb02-7889a4a780ce/7dcf5a40-78e3-4718-8bc4-f9cdc266173a"
+					(reference "J2")
+					(unit 1)
+				)
+				(path "/2e03126f-90c3-49c2-bb02-7889a4a780ce/a445d34f-af0c-4abc-8750-cad3f5a4f178"
+					(reference "J13")
+					(unit 1)
+				)
+				(path "/2e03126f-90c3-49c2-bb02-7889a4a780ce/e44134ae-6fd5-457c-b7e1-8d10f2737c1e"
+					(reference "J15")
+					(unit 1)
+				)
+				(path "/2e03126f-90c3-49c2-bb02-7889a4a780ce/f4b37abd-93fa-47ac-8113-341753863783"
+					(reference "J11")
+					(unit 1)
+				)
