File: PT100.kicad_sch (KiCad schematic)
At the start: 4 parts, among them IC3 MAX31865ATP+T

Commit message: Added stuff
Parts:
- added J3: B4B-XH-A_LF__SN_, B4BXHALFSN, symbol B4B-XH-A_LF__SN_:B4B-XH-A_LF__SN_
- IC3: footprint QFN65P500X500X80-21N -> Library:QFN65P500X500X80-21N
- S1: footprint 2194MST -> Library:2194MST
- renumbered R12 to R10, R13 to R11
Connections:
- net 4300R: now also R11.1
- net 430R: now also R10.1
- net FORCE_N: now also J3.1
- net FORCE_P: now also J3.4
- net RTDIN_N: now also J3.2
- net RTDIN_P: now also J3.3
Other:
- moved on the sheet: IC3, R10, R11, S1

Commit message: small changes
Parts:
- removed J3: B4B-XH-A_LF__SN_, B4BXHALFSN, symbol B4B-XH-A_LF__SN_:B4B-XH-A_LF__SN_
- added J4: 691412120004B, Library:691412120004B, symbol 691412120004B:691412120004B
- renumbered IC3 to IC7, R10 to R27, R11 to R28, S1 to S2
Connections:
- net FORCE_N: now also J4.4
- net FORCE_P: now also J4.1
- net RTDIN_N: now also J4.3
- net RTDIN_P: now also J4.2

Commit message: lots of change
Parts:
- removed IC7: MAX31865ATP+T, Library:QFN65P500X500X80-21N, symbol MAX31865ATP+T:MAX31865ATP+T
- removed J4: 691412120004B, Library:691412120004B, symbol 691412120004B:691412120004B
- added IC4: MAX31865ATP+T, QFN65P500X500X80-21N, symbol afterburner_symbolic:MAX31865ATP+T
- added J17: 1803293, Library:PHOENIX_1803293, symbol afterburner_symbolic:1803293
Connections:
- net +3V3: now also IC4.19 (DVDD), IC4.20 (VDD)
- net CS: now also IC4.13 (~{CS})
- net FORCE_N: now also IC4.9 (FORCE-), J17.04
- net FORCE_P: now also IC4.5 (FORCE+), J17.01
- net GND: now also IC4.10 (GND2), IC4.15 (DGND), IC4.16 (GND1), IC4.21 (EP), IC4.6 (FORCE2)
- net ISENSOR: now also IC4.3 (REFIN-), IC4.4 (ISENSOR)
- net MISO: now also IC4.14 (SDO)
- net MOSI: now also IC4.11 (SDI)
- net RTDIN_N: now also IC4.8 (RTDIN-), J17.03
- net RTDIN_P: now also IC4.7 (RTDIN+), J17.02
- net SCLK: now also IC4.12 (SCLK)
- net at R27.2, R28.2: now also IC4.1 (BIAS), IC4.2 (REFIN+)
