File: loadcell.kicad_sch (KiCad schematic)
At the start: 5 parts, among them IC4 ADS131M02IRUKR, J4 B4B-XH-A_LF__SN_

Commit message: Added stuff
Parts:
- removed IC4: ADS131M02IRUKR, QFN40P300X300X80-21N-D, symbol ADS131M02IRUKR:ADS131M02IRUKR
- added C8: 1uF, Capacitor_SMD:C_0402_1005Metric, symbol Device:C
- added IC4: NAU7802SGI, SOIC127P600X175-16N, symbol NAU7802SGI:NAU7802SGI
- C5: value 220nF -> 1uF
- C6, C7: footprint (none) -> Capacitor_SMD:C_0402_1005Metric
- J4: footprint B4BXHALFSN -> Library:B4BXHALFSN
Connections:
- net +3V3: now also IC4.15 (DVDD); no longer C6.1, C7.1
- net GND: now also J4.3, C8.2, IC4.7 (REFN), IC4.8 (AVSS), IC4.9 (DVSS); no longer C6.2
- net SCLK: now also IC4.13 (SCLK)
- net at C5.1: now also J4.4, C8.1, IC4.1 (REFP), IC4.16 (AVDD/LDO)
- net at J4.1: now also IC4.3 (VIN1P)
- net at J4.2: now also IC4.2 (VIN1N)
- new net: C6.1, IC4.4 (VIN2N)
- new net: C6.2, IC4.5 (VIN2P)
- new net: C7.1, IC4.6 (VBG)
- new net DRDY: IC4.12 (DRDY)
- new net SDIO: IC4.14 (SDIO)
- no-connect marks 4 -> 2
Other:
- moved on the sheet: J4

Commit message: small changes
Parts:
- removed J4: B4B-XH-A_LF__SN_, Library:B4BXHALFSN, symbol B4B-XH-A_LF__SN_:B4B-XH-A_LF__SN_
- added J3: 691412120004B, Library:691412120004B, symbol 691412120004B:691412120004B
- renumbered IC4 to IC3
Connections:
- net GND: now also J3.2
- net at C5.1, C8.1, IC3.1 (REFP)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: now also J3.1
- net at IC3.2 (VIN1N): now also J3.3
- net at IC3.3 (VIN1P): now also J3.4
Changed lines of the file:
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@@
+	(wire
+		(pts
+			(xy 58.42 64.77) (xy 82.55 64.77)
+		)
+		(stroke
+			(width 0)
+			(type default)
+		)
+	)
 	(wire
 		(pts
@@
 	(wire
 		(pts
+			(xy 68.58 62.23) (xy 82.55 62.23)
+		)
+		(stroke
+			(width 0)
+			(type default)
+		)
+	)
+	(wire
+		(pts
 			(xy 111.76 44.45) (xy 147.32 44.45)
 		)
@@
 	(wire
 		(pts
-			(xy 74.93 62.23) (xy 82.55 62.23)
-		)
-		(stroke
-			(width 0)
-			(type default)
-		)
-	)
-	(wire
-		(pts
 			(xy 116.84 78.74) (xy 116.84 86.36)
 		)
@@
 	(wire
 		(pts
-			(xy 88.9 67.31) (xy 74.93 67.31)
-		)
-		(stroke
-			(width 0)
-			(type default)
-		)
-	)
-	(wire
-		(pts
 			(xy 97.79 74.93) (xy 102.87 74.93)
 		)
@@
 	(wire
 		(pts
+			(xy 58.42 69.85) (xy 91.44 69.85)
+		)
+		(stroke
+			(width 0)
+			(type default)
+		)
+	)
+	(wire
+		(pts
 			(xy 106.68 81.28) (xy 106.68 86.36)
 		)
@@
 	(wire
 		(pts
+			(xy 68.58 67.31) (xy 88.9 67.31)
+		)
+		(stroke
+			(width 0)
+			(type default)
+		)
+	)
+	(wire
+		(pts
 			(xy 116.84 86.36) (xy 116.84 90.17)
 		)
@@
 	(wire
 		(pts
-			(xy 82.55 64.77) (xy 74.93 64.77)
-		)
-		(stroke
-			(width 0)
-			(type default)
-		)
-	)
-	(wire
-		(pts
 			(xy 91.44 69.85) (xy 91.44 66.04)
 		)
@@
 		(pts
 			(xy 82.55 44.45) (xy 96.52 44.45)
-		)
-		(stroke
-			(width 0)
-			(type default)
-		)
-	)
-	(wire
-		(pts
-			(xy 74.93 69.85) (xy 91.44 69.85)
 		)
 		(stroke
@@
 		(dnp no)
 		(fields_autoplaced yes)
-		(property "Reference" "IC4"
+		(property "Reference" "IC3"
 			(at 134.62 53.34 0)
 			(effects
@@
 			(project ""
 				(path "/2e03126f-90c3-49c2-bb02-7889a4a780ce/d4aa8317-4dd0-460d-8e3e-edb5da807fd1"
-					(reference "IC4")
+					(reference "IC3")
 					(unit 1)
 				)
@@
 		(dnp no)
 		(fields_autoplaced yes)
-		(property "Reference" "#PWR023"
+		(property "Reference" "#PWR017"
 			(at 116.84 96.52 0)
 			(effects
@@
 			(project ""
 				(path "/2e03126f-90c3-49c2-bb02-7889a4a780ce/d4aa8317-4dd0-460d-8e3e-edb5da807fd1"
-					(reference "#PWR023")
+					(reference "#PWR017")
+					(unit 1)
+				)
+			)
+		)
+	)
+	(symbol
+		(lib_id "691412120004B:691412120004B")
+		(at 63.5 64.77 90)
+		(mirror x)
+		(unit 1)
+		(exclude_from_sim no)
+		(in_bom yes)
+		(on_board yes)
+		(dnp no)
+		(property "Reference" "J3"
+			(at 63.5 76.2 90)
+			(effects
+				(font
+					(size 1.27 1.27)
+				)
+			)
+		)
+		(property "Value" "691412120004B"
+			(at 63.5 73.66 90)
+			(effects
+				(font
+					(size 1.27 1.27)
+				)
+			)
+		)
+		(property "Footprint" "Library:691412120004B"
+			(at 63.5 64.77 0)
+			(effects
+				(font
+					(size 1.27 1.27)
+				)
+				(justify bottom)
+				(hide yes)
+			)
+		)
+		(property "Datasheet" ""
+			(at 63.5 64.77 0)
+			(effects
+				(font
+					(size 1.27 1.27)
+				)
+				(hide yes)
+			)
+		)
+		(property "Description" ""
+			(at 63.5 64.77 0)
+			(effects
+				(font
+					(size 1.27 1.27)
+				)
+				(hide yes)
+			)
+		)
+		(pin "2"
+		)
+		(pin "3"
+		)
+		(pin "1"
+		)
+		(pin "4"
+		)
+		(instances
+			(project "first_project"
+				(path "/2e03126f-90c3-49c2-bb02-7889a4a780ce/d4aa8317-4dd0-460d-8e3e-edb5da807fd1"
+					(reference "J3")
 					(unit 1)
 				)
@@
 		(dnp no)
 		(fields_autoplaced yes)
-		(property "Reference" "#PWR024"
+		(property "Reference" "#PWR018"
 			(at 147.32 58.42 0)
 			(effects
@@
 			(project ""
 				(path "/2e03126f-90c3-49c2-bb02-7889a4a780ce/d4aa8317-4dd0-460d-8e3e-edb5da807fd1"
-					(reference "#PWR024")
+					(reference "#PWR018")
 					(unit 1)
 				)
@@
 		(dnp no)
 		(fields_autoplaced yes)
-		(property "Reference" "#PWR022"
+		(property "Reference" "#PWR016"
 			(at 96.52 58.42 0)
 			(effects
@@
 			(project "first_project"
 				(path "/2e03126f-90c3-49c2-bb02-7889a4a780ce/d4aa8317-4dd0-460d-8e3e-edb5da807fd1"
-					(reference "#PWR022")
+					(reference "#PWR016")
 					(unit 1)
 				)
@@
 		(dnp no)
 		(fields_autoplaced yes)
-		(property "Reference" "#PWR025"
+		(property "Reference" "#PWR019"
 			(at 160.02 49.53 0)
 			(effects
@@
 			(project ""
 				(path "/2e03126f-90c3-49c2-bb02-7889a4a780ce/d4aa8317-4dd0-460d-8e3e-edb5da807fd1"
-					(reference "#PWR025")
+					(reference "#PWR019")
 					(unit 1)
 				)
-			)
-		)
-	)
-	(symbol
-		(lib_id "B4B-XH-A_LF__SN_:B4B-XH-A_LF__SN_")
-		(at 74.93 69.85 180)
-		(unit 1)
-		(exclude_from_sim no)
-		(in_bom yes)
-		(on_board yes)
-		(dnp no)
-		(fields_autoplaced yes)
-		(property "Reference" "J4"
-			(at 64.77 54.61 0)
-			(effects
-				(font
-					(size 1.27 1.27)
-				)
-			)
-		)
-		(property "Value" "B4B-XH-A_LF__SN_"
-			(at 64.77 57.15 0)
-			(effects
-				(font
-					(size 1.27 1.27)
-				)
-			)
-		)
-		(property "Footprint" "Library:B4BXHALFSN"
-			(at 58.42 -25.07 0)
-			(effects
-				(font
-					(size 1.27 1.27)
-				)
-				(justify left top)
-				(hide yes)
-			)
-		)
-		(property "Datasheet" "https://datasheet.lcsc.com/szlcsc/JST-Sales-America-B4B-XH-A-LF-SN_C144395.pdf"
-			(at 58.42 -125.07 0)
-			(effects
-				(font
-					(size 1.27 1.27)
-				)
-				(justify left top)
-				(hide yes)
-			)
-		)
-		(property "Description" "CONN HEADER VERT 4POS 2.5MM"
-			(at 74.93 69.85 0)
-			(effects
-				(font
-					(size 1.27 1.27)
-				)
-				(hide yes)
-			)
-		)
-		(property "Height" "7"
-			(at 58.42 -325.07 0)
-			(effects
-				(font
-					(size 1.27 1.27)
-				)
-				(justify left top)
-				(hide yes)
-			)
-		)
-		(property "Mouser Part Number" "306-B4BXHALFSN"
-			(at 58.42 -425.07 0)
-			(effects
-				(font
-					(size 1.27 1.27)
-				)
-				(justify left top)
-				(hide yes)
-			)
-		)
-		(property "Mouser Price/Stock" "https://www.mouser.co.uk/ProductDetail/JST-Commercial/B4B-XH-ALFSN?qs=cdbOS8ANM9CfC08d%252BywhFw%3D%3D"
-			(at 58.42 -525.07 0)
-			(effects
-				(font
-					(size 1.27 1.27)
-				)
-				(justify left top)
-				(hide yes)
-			)
-		)
-		(property "Manufacturer_Name" "JST (JAPAN SOLDERLESS TERMINALS)"
-			(at 58.42 -625.07 0)
-			(effects
-				(font
-					(size 1.27 1.27)
-				)
-				(justify left top)
-				(hide yes)
-			)
-		)
-		(property "Manufacturer_Part_Number" "B4B-XH-A(LF)(SN)"
-			(at 58.42 -725.07 0)
-			(effects
-				(font
-					(size 1.27 1.27)
-				)
-				(justify left top)
-				(hide yes)
-			)
-		)
-		(pin "3"
-		)
-		(pin "2"
-		)
-		(pin "4"
-		)
-		(pin "1"
-		)
-		(instances
-			(project ""
-				(path "/2e03126f-90c3-49c2-bb02-7889a4a780ce/d4aa8317-4dd0-460d-8e3e-edb5da807fd1"
-					(reference "J4")
-					(unit 1)
-				)

Commit message: changes
Parts:
- IC3: footprint SOIC127P600X175-16N -> Library:SOIC127P600X175-16N
Changed lines of the file:
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@@
 			)
 		)
-		(property "Footprint" "SOIC127P600X175-16N"
+		(property "Footprint" "Library:SOIC127P600X175-16N"
 			(at 148.59 155.88 0)
 			(effects

Commit message: lots of change
Parts:
- removed J3: 691412120004B, Library:691412120004B, symbol 691412120004B:691412120004B
- added J3: 1803293, Library:PHOENIX_1803293, symbol afterburner_symbolic:1803293
Connections:
- net GND: now also J3.02
- net at C5.1, C8.1, IC3.1 (REFP)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: now also J3.01
- net at IC3.2 (VIN1N): now also J3.03
- net at IC3.3 (VIN1P): now also J3.04
Changed lines of the file:
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@@
+	(wire
+		(pts
+			(xy 58.42 62.23) (xy 82.55 62.23)
+		)
+		(stroke
+			(width 0)
+			(type default)
+		)
+	)
 	(wire
 		(pts
@@
 	(wire
 		(pts
-			(xy 68.58 62.23) (xy 82.55 62.23)
-		)
-		(stroke
-			(width 0)
-			(type default)
-		)
-	)
-	(wire
-		(pts
 			(xy 111.76 44.45) (xy 147.32 44.45)
 		)
@@
 	(wire
 		(pts
-			(xy 68.58 67.31) (xy 88.9 67.31)
-		)
-		(stroke
-			(width 0)
-			(type default)
-		)
-	)
-	(wire
-		(pts
 			(xy 116.84 86.36) (xy 116.84 90.17)
 		)
@@
 		(pts
 			(xy 91.44 69.85) (xy 91.44 66.04)
+		)
+		(stroke
+			(width 0)
+			(type default)
+		)
+	)
+	(wire
+		(pts
+			(xy 58.42 67.31) (xy 88.9 67.31)
 		)
 		(stroke
@@
 	)
 	(symbol
+		(lib_id "afterburner_symbolic:1803293")
+		(at 48.26 67.31 0)
+		(mirror y)
+		(unit 1)
+		(exclude_from_sim no)
+		(in_bom yes)
+		(on_board yes)
+		(dnp no)
+		(property "Reference" "J3"
+			(at 48.26 77.47 0)
+			(effects
+				(font
+					(size 1.27 1.27)
+				)
+			)
+		)
+		(property "Value" "1803293"
+			(at 48.26 74.93 0)
+			(effects
+				(font
+					(size 1.27 1.27)
+				)
+			)
+		)
+		(property "Footprint" "Library:PHOENIX_1803293"
+			(at 48.26 67.31 0)
+			(effects
+				(font
+					(size 1.27 1.27)
+				)
+				(justify bottom)
+				(hide yes)
+			)
+		)
+		(property "Datasheet" ""
+			(at 48.26 67.31 0)
+			(effects
+				(font
+					(size 1.27 1.27)
+				)
+				(hide yes)
+			)
+		)
+		(property "Description" ""
+			(at 48.26 67.31 0)
+			(effects
+				(font
+					(size 1.27 1.27)
+				)
+				(hide yes)
+			)
+		)
+		(property "PARTREV" "08.06.2015"
+			(at 48.26 67.31 0)
+			(effects
+				(font
+					(size 1.27 1.27)
+				)
+				(justify bottom)
+				(hide yes)
+			)
+		)
+		(property "STANDARD" "Manufacturer Recommendations"
+			(at 48.26 67.31 0)
+			(effects
+				(font
+					(size 1.27 1.27)
+				)
+				(justify bottom)
+				(hide yes)
+			)
+		)
+		(property "MANUFACTURER" "Phoenix Contact"
+			(at 48.26 67.31 0)
+			(effects
+				(font
+					(size 1.27 1.27)
+				)
+				(justify bottom)
+				(hide yes)
+			)
+		)
+		(pin "03"
+		)
+		(pin "04"
+		)
+		(pin "02"
+		)
+		(pin "01"
+		)
+		(instances
+			(project "afterburner"
+				(path "/2e03126f-90c3-49c2-bb02-7889a4a780ce/d4aa8317-4dd0-460d-8e3e-edb5da807fd1"
+					(reference "J3")
+					(unit 1)
+				)
+			)
+		)
+	)
+	(symbol
 		(lib_id "Device:C")
 		(at 106.68 77.47 0)
@@
 					(unit 1)
 				)
-			)
-		)
-	)
-	(symbol
-		(lib_id "691412120004B:691412120004B")
-		(at 63.5 64.77 90)
-		(mirror x)
-		(unit 1)
-		(exclude_from_sim no)
-		(in_bom yes)
-		(on_board yes)
-		(dnp no)
-		(property "Reference" "J3"
-			(at 63.5 76.2 90)
-			(effects
-				(font
-					(size 1.27 1.27)
-				)
-			)
-		)
-		(property "Value" "691412120004B"
-			(at 63.5 73.66 90)
-			(effects
-				(font
-					(size 1.27 1.27)
-				)
-			)
-		)
-		(property "Footprint" "Library:691412120004B"
-			(at 63.5 64.77 0)
-			(effects
-				(font
-					(size 1.27 1.27)
-				)
-				(justify bottom)
-				(hide yes)
-			)
-		)
-		(property "Datasheet" ""
-			(at 63.5 64.77 0)
-			(effects
-				(font
-					(size 1.27 1.27)
-				)
-				(hide yes)
-			)
-		)
-		(property "Description" ""
-			(at 63.5 64.77 0)
-			(effects
-				(font
-					(size 1.27 1.27)
-				)
-				(hide yes)
-			)
-		)
-		(pin "2"
-		)
-		(pin "3"
-		)
-		(pin "1"
-		)
-		(pin "4"
-		)
-		(instances
-			(project "first_project"
-				(path "/2e03126f-90c3-49c2-bb02-7889a4a780ce/d4aa8317-4dd0-460d-8e3e-edb5da807fd1"
-					(reference "J3")
-					(unit 1)
-				)
